Commit message: Changed tool_0 to tool0. Fixed numerical artifacts and centered all joints on the xz plane

File: abb_irb2600_support/urdf/irb2600_macro.xacro (robot description, xacro)
@@ -38,5 +38,5 @@
     </link>
     <joint name="${prefix}joint_1" type="revolute">
-      <origin xyz="1.0538E-05 0 0.20551" rpy="0 0 0" />
+      <origin xyz="0.0 0 0.20551" rpy="0 0 0" />
       <parent link="${prefix}base_link" />
       <child link="${prefix}link_1" />
@@ -46,5 +46,5 @@
     <link name="${prefix}link_2">
       <visual>
-        <origin xyz="0 0 0" rpy="0 0 0" />
+        <origin xyz="0 -0.1524 0" rpy="0 0 0" />
         <geometry>
           <mesh filename="package://abb_irb2600_support/meshes/visual/link_2.STL" />
@@ -55,5 +55,5 @@
       </visual>
       <collision>
-        <origin xyz="0 0 0" rpy="0 0 0" />
+        <origin xyz="0 -0.1524 0" rpy="0 0 0" />
         <geometry>
           <mesh filename="package://abb_irb2600_support/meshes/collision/link_2.STL" />
@@ -62,5 +62,5 @@
     </link>
     <joint name="${prefix}joint_2" type="revolute">
-      <origin xyz="0.14999 -0.1524 0.23949" rpy="0 0 0" />
+      <origin xyz="0.14999 0.0 0.23949" rpy="0 0 0" />
       <parent link="${prefix}link_1" />
       <child link="${prefix}link_2" />
@@ -70,5 +70,5 @@
     <link name="${prefix}link_3">
       <visual>
-        <origin xyz="0 0 0" rpy="0 0 0" />
+        <origin xyz="0 ${0.0046 - 0.1524}  0" rpy="0 0 0" />
         <geometry>
           <mesh filename="package://abb_irb2600_support/meshes/visual/link_3.STL" />
@@ -79,5 +79,5 @@
       </visual>
       <collision>
-        <origin xyz="0 0 0" rpy="0 0 0" />
+        <origin xyz="0 ${0.0046 - 0.1524} 0" rpy="0 0 0" />
         <geometry>
           <mesh filename="package://abb_irb2600_support/meshes/collision/link_3.STL" />
@@ -86,5 +86,5 @@
     </link>
     <joint name="${prefix}joint_3" type="revolute">
-      <origin xyz="0 0.0046 0.7" rpy="0 0 0" />
+      <origin xyz="0 0.0 0.7" rpy="0 0 0" />
       <parent link="${prefix}link_2" />
       <child link="${prefix}link_3" />
@@ -94,5 +94,5 @@
     <link name="${prefix}link_4">
       <visual>
-        <origin xyz="0 0 0" rpy="0 0 0" />
+        <origin xyz="0 ${0.1478 + 0.0046 - 0.1524} 0" rpy="0 0 0" />
         <geometry>
           <mesh filename="package://abb_irb2600_support/meshes/visual/link_4.STL" />
@@ -103,5 +103,5 @@
       </visual>
       <collision>
-        <origin xyz="0 0 0" rpy="0 0 0" />
+        <origin xyz="0 ${0.1478 + 0.0046 - 0.1524} 0" rpy="0 0 0" />
         <geometry>
           <mesh filename="package://abb_irb2600_support/meshes/collision/link_4.STL" />
@@ -110,5 +110,5 @@
     </link>
     <joint name="${prefix}joint_4" type="revolute">
-      <origin xyz="0.288 0.1478 0.115" rpy="0 0 0" />
+      <origin xyz="0.288 0.0 0.115" rpy="0 0 0" />
       <parent link="${prefix}link_3" />
       <child link="${prefix}link_4" />
@@ -134,5 +134,5 @@
     </link>
     <joint name="${prefix}joint_5" type="revolute">
-      <origin xyz="0.50733 -0.0020554 -0.00011374" rpy="0 0 0" />
+      <origin xyz="0.50733 0.0 0.0" rpy="0 0 0" />
       <parent link="${prefix}link_4" />
       <child link="${prefix}link_5" />
@@ -158,5 +158,5 @@
     </link>
     <joint name="${prefix}joint_6" type="revolute">
-      <origin xyz="0.056713 5.5386E-05 0.00011374" rpy="0 0 0" />
+      <origin xyz="0.056713 0.0 0.0" rpy="0 0 0" />
       <parent link="${prefix}link_5" />
       <child link="${prefix}link_6" />
@@ -164,9 +164,9 @@
       <limit lower="-6.981" upper="6.981" effort="0" velocity="8.727" />
     </joint>
-    <link name="${prefix}tool_0" />
+    <link name="${prefix}tool0" />
     <joint name="${prefix}joint_t0" type="fixed">
-      <origin xyz="0.025958 0 0" rpy="0 0 0" />
+      <origin xyz="0.025958 0 0" rpy="0 1.5707963267948966 0" />
       <parent link="${prefix}link_6" />
-      <child link="${prefix}tool_0" />
+      <child link="${prefix}tool0" />
       <axis xyz="0 0 0" />
       <limit lower="-1" upper="1" effort="0" velocity="1" />

Commit message: Updated 2600 urdf

File: abb_irb2600_support/urdf/irb2600_macro.xacro (robot description, xacro)
@@ -1,181 +1,323 @@
-<?xml version="1.0" encoding="UTF-8"?>
+<?xml version="1.0" ?>
 <robot xmlns:xacro="http://ros.org/wiki/xacro">
   <xacro:macro name="abb_irb2600" params="prefix">
-    <!-- links -->
-    <link name="${prefix}base_link">
-      <visual>
-        <origin xyz="0 0 0" rpy="0 0 0" />
-        <geometry>
-          <mesh filename="package://abb_irb2600_support/meshes/visual/base_link.STL" />
-        </geometry>
-        <material name="">
-          <color rgba="1 0.50196 0 1" />
-        </material>
-      </visual>
-      <collision>
-        <origin xyz="0 0 0" rpy="0 0 0" />
-        <geometry>
-          <mesh filename="package://abb_irb2600_support/meshes/collision/base_link.STL" />
-        </geometry>
-      </collision>
-    </link>
-    <link name="${prefix}link_1">
-      <visual>
-        <origin xyz="0 0 0" rpy="0 0 0" />
-        <geometry>
-          <mesh filename="package://abb_irb2600_support/meshes/visual/link_1.STL" />
-        </geometry>
-        <material name="">
-          <color rgba="1 0.50196 0 1" />
-        </material>
-      </visual>
-      <collision>
-        <origin xyz="0 0 0" rpy="0 0 0" />
-        <geometry>
-          <mesh filename="package://abb_irb2600_support/meshes/collision/link_1.STL" />
-        </geometry>
-      </collision>
-    </link>
-    <joint name="${prefix}joint_1" type="revolute">
-      <origin xyz="0.0 0 0.20551" rpy="0 0 0" />
-      <parent link="${prefix}base_link" />
-      <child link="${prefix}link_1" />
-      <axis xyz="0 0 1" />
-      <limit lower="-3.14159" upper="3.14159" effort="0" velocity="3.054" />
-    </joint>
-    <link name="${prefix}link_2">
-      <visual>
-        <origin xyz="0 -0.1524 0" rpy="0 0 0" />
-        <geometry>
-          <mesh filename="package://abb_irb2600_support/meshes/visual/link_2.STL" />
-        </geometry>
-        <material name="">
-          <color rgba="1 0.50196 0 1" />
-        </material>
-      </visual>
-      <collision>
-        <origin xyz="0 -0.1524 0" rpy="0 0 0" />
-        <geometry>
-          <mesh filename="package://abb_irb2600_support/meshes/collision/link_2.STL" />
-        </geometry>
-      </collision>
-    </link>
-    <joint name="${prefix}joint_2" type="revolute">
-      <origin xyz="0.14999 0.0 0.23949" rpy="0 0 0" />
-      <parent link="${prefix}link_1" />
-      <child link="${prefix}link_2" />
-      <axis xyz="0 -1 0" />
-      <limit lower="-2.705" upper="1.658" effort="0" velocity="3.054" />
-    </joint>
-    <link name="${prefix}link_3">
-      <visual>
-        <origin xyz="0 ${0.0046 - 0.1524}  0" rpy="0 0 0" />
-        <geometry>
-          <mesh filename="package://abb_irb2600_support/meshes/visual/link_3.STL" />
-        </geometry>
-        <material name="">
-          <color rgba="1 0.50196 0 1" />
-        </material>
-      </visual>
-      <collision>
-        <origin xyz="0 ${0.0046 - 0.1524} 0" rpy="0 0 0" />
-        <geometry>
-          <mesh filename="package://abb_irb2600_support/meshes/collision/link_3.STL" />
-        </geometry>
-      </collision>
-    </link>
-    <joint name="${prefix}joint_3" type="revolute">
-      <origin xyz="0 0.0 0.7" rpy="0 0 0" />
-      <parent link="${prefix}link_2" />
-      <child link="${prefix}link_3" />
-      <axis xyz="0 1 0" />
-      <limit lower="-2.705" upper="1.309" effort="0" velocity="3.054" />
-    </joint>
-    <link name="${prefix}link_4">
-      <visual>
-        <origin xyz="0 ${0.1478 + 0.0046 - 0.1524} 0" rpy="0 0 0" />
-        <geometry>
-          <mesh filename="package://abb_irb2600_support/meshes/visual/link_4.STL" />
-        </geometry>
-        <material name="">
-          <color rgba="1 0.50196 0 1" />
-        </material>
-      </visual>
-      <collision>
-        <origin xyz="0 ${0.1478 + 0.0046 - 0.1524} 0" rpy="0 0 0" />
-        <geometry>
-          <mesh filename="package://abb_irb2600_support/meshes/collision/link_4.STL" />
-        </geometry>
-      </collision>
-    </link>
-    <joint name="${prefix}joint_4" type="revolute">
-      <origin xyz="0.288 0.0 0.115" rpy="0 0 0" />
-      <parent link="${prefix}link_3" />
-      <child link="${prefix}link_4" />
-      <axis xyz="-1 0 0" />
-      <limit lower="-6.981" upper="6.981" effort="0" velocity="6.283" />
-    </joint>
-    <link name="${prefix}link_5">
-      <visual>
-        <origin xyz="0 0 0" rpy="0 0 0" />
-        <geometry>
-          <mesh filename="package://abb_irb2600_support/meshes/visual/link_5.STL" />
-        </geometry>
-        <material name="">
-          <color rgba="1 0.50196 0 1" />
-        </material>
-      </visual>
-      <collision>
-        <origin xyz="0 0 0" rpy="0 0 0" />
-        <geometry>
-          <mesh filename="package://abb_irb2600_support/meshes/collision/link_5.STL" />
-        </geometry>
-      </collision>
-    </link>
-    <joint name="${prefix}joint_5" type="revolute">
-      <origin xyz="0.50733 0.0 0.0" rpy="0 0 0" />
-      <parent link="${prefix}link_4" />
-      <child link="${prefix}link_5" />
-      <axis xyz="0 1 0" />
-      <limit lower="-2.094" upper="2.094" effort="0" velocity="6.283" />
-    </joint>
-    <link name="${prefix}link_6">
-      <visual>
-        <origin xyz="0 0 0" rpy="0 0 0" />
-        <geometry>
-          <mesh filename="package://abb_irb2600_support/meshes/visual/link_6.STL" />
-        </geometry>
-        <material name="">
-          <color rgba="0.49804 0.49804 0.49804 1" />
-        </material>
-      </visual>
-      <collision>
-        <origin xyz="0 0 0" rpy="0 0 0" />
-        <geometry>
-          <mesh filename="package://abb_irb2600_support/meshes/collision/link_6.STL" />
-        </geometry>
-      </collision>
-    </link>
-    <joint name="${prefix}joint_6" type="revolute">
-      <origin xyz="0.056713 0.0 0.0" rpy="0 0 0" />
-      <parent link="${prefix}link_5" />
-      <child link="${prefix}link_6" />
-      <axis xyz="1 0 0" />
-      <limit lower="-6.981" upper="6.981" effort="0" velocity="8.727" />
-    </joint>
-    <link name="${prefix}tool0" />
-    <joint name="${prefix}joint_t0" type="fixed">
-      <origin xyz="0.025958 0 0" rpy="0 1.5707963267948966 0" />
-      <parent link="${prefix}link_6" />
-      <child link="${prefix}tool0" />
-      <axis xyz="0 0 0" />
-      <limit lower="-1" upper="1" effort="0" velocity="1" />
-    </joint>
-    <link name="${prefix}base" />
-    <joint name="${prefix}base_link-base" type="fixed">
-      <origin xyz="0 0 0.450" rpy="0 0 0" />
-      <parent link="${prefix}base_link" />
-      <child link="${prefix}base" />
-    </joint>
-  </xacro:macro>
-</robot>
+     <!-- links -->
+<link
+    name="${prefix}base_link">
+    <visual>
+      <origin
+        xyz="0 0 0"
+        rpy="0 0 0" />
+      <geometry>
+        <mesh
+          filename="package://abb_irb2600_support/meshes/visual/base_link.STL" />
+      </geometry>
+      <material
+        name="">
+        <color
+          rgba="1 0.50196 0 1" />
+      </material>
+    </visual>
+    <collision>
+      <origin
+        xyz="0 0 0"
+        rpy="0 0 0" />
+      <geometry>
+        <mesh
+          filename="package://abb_irb2600_support/meshes/collision/base_link.STL" />
+      </geometry>
+    </collision>
+  </link>
+  <link
+    name="${prefix}link_1">
+    <visual>
+      <origin
+        xyz="0 0 0"
+        rpy="0 0 0" />
+      <geometry>
+        <mesh
+          filename="package://abb_irb2600_support/meshes/visual/link_1.STL" />
+      </geometry>
+      <material
+        name="">
+        <color
+          rgba="1 0.50196 0 1" />
+      </material>
+    </visual>
+    <collision>
+      <origin
+        xyz="0 0 0"
+        rpy="0 0 0" />
+      <geometry>
+        <mesh
+          filename="package://abb_irb2600_support/meshes/collision/link_1.STL" />
+      </geometry>
+    </collision>
+  </link>
+  <joint
+    name="${prefix}joint_1"
+    type="revolute">
+    <origin
+      xyz="0 0 0.20551"
+      rpy="0 0 0" />
+    <parent
+      link="${prefix}base_link" />
+    <child
+      link="${prefix}link_1" />
+    <axis
+      xyz="0 0 1" />
+    <limit
+      lower="-3.14159"
+      upper="3.14159"
+      effort="0"
+      velocity="3.054" />
+  </joint>
+  <link
+    name="${prefix}link_2">
+    <visual>
+      <origin
+        xyz="0 0 0"
+        rpy="0 0 0" />
+      <geometry>
+        <mesh
+          filename="package://abb_irb2600_support/meshes/visual/link_2.STL" />
+      </geometry>
+      <material
+        name="">
+        <color
+          rgba="1 0.50196 0 1" />
+      </material>
+    </visual>
+    <collision>
+      <origin
+        xyz="0 0 0"
+        rpy="0 0 0" />
+      <geometry>
+        <mesh
+          filename="package://abb_irb2600_support/meshes/collision/link_2.STL" />
+      </geometry>
+    </collision>
+  </link>
+  <joint
+    name="${prefix}joint_2"
+    type="revolute">
+    <origin
+      xyz="0.14999 0 0.23949"
+      rpy="0 0 0" />
+    <parent
+      link="${prefix}link_1" />
+    <child
+      link="${prefix}link_2" />
+    <axis
+      xyz="0 -1 0" />
+    <limit
+      lower="-2.705"
+      upper="1.658"
+      effort="0"
+      velocity="3.054" />
+  </joint>
+  <link
+    name="${prefix}link_3">
+    <visual>
+      <origin
+        xyz="0 0 0"
+        rpy="0 0 0" />
+      <geometry>
+        <mesh
+          filename="package://abb_irb2600_support/meshes/visual/link_3.STL" />
+      </geometry>
+      <material
+        name="">
+        <color
+          rgba="1 0.50196 0 1" />
+      </material>
+    </visual>
+    <collision>
+      <origin
+        xyz="0 0 0"
+        rpy="0 0 0" />
+      <geometry>
+        <mesh
+          filename="package://abb_irb2600_support/meshes/collision/link_3.STL" />
+      </geometry>
+    </collision>
+  </link>
+  <joint
+    name="${prefix}joint_3"
+    type="revolute">
+    <origin
+      xyz="0 0 0.7"
+      rpy="0 0 0" />
+    <parent
+      link="${prefix}link_2" />
+    <child
+      link="${prefix}link_3" />
+    <axis
+      xyz="0 1 0" />
+    <limit
+      lower="-2.705"
+      upper="1.309"
+      effort="0"
+      velocity="3.054" />
+  </joint>
+  <link
+    name="${prefix}link_4">
+    <visual>
+      <origin
+        xyz="0 0 0"
+        rpy="0 0 0" />
+      <geometry>
+        <mesh
+          filename="package://abb_irb2600_support/meshes/visual/link_4.STL" />
+      </geometry>
+      <material
+        name="">
+        <color
+          rgba="1 0.50196 0 1" />
+      </material>
+    </visual>
+    <collision>
+      <origin
+        xyz="0 0 0"
+        rpy="0 0 0" />
+      <geometry>
+        <mesh
+          filename="package://abb_irb2600_support/meshes/collision/link_4.STL" />
+      </geometry>
+    </collision>
+  </link>
+  <joint
+    name="${prefix}joint_4"
+    type="revolute">
+    <origin
+      xyz="0.288 0 0.115"
+      rpy="0 0 0" />
+    <parent
+      link="${prefix}link_3" />
+    <child
+      link="${prefix}link_4" />
+    <axis
+      xyz="-1 0 0" />
+    <limit
+      lower="-6.981"
+      upper="6.981"
+      effort="0"
+      velocity="6.283" />
+  </joint>
+  <link
+    name="${prefix}link_5">
+    <visual>
+      <origin
+        xyz="0 0 0"
+        rpy="0 0 0" />
+      <geometry>
+        <mesh
+          filename="package://abb_irb2600_support/meshes/visual/link_5.STL" />
+      </geometry>
+      <material
+        name="">
+        <color
+          rgba="1 0.50196 0 1" />
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