Commit message: Major adjustments for the particular robot we are using

File: abb_irb6600_support/urdf/irb6600.urdf (robot description, URDF)
Before this commit: robot None, 0 links, 0 joints
Links:
- added link base
- added link base_link; collision mesh filename=package://abb_irb6600_support/meshes/irb6600_225_255/collis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; visual mesh filename=package://abb_irb6600_support/meshes/irb6600_225_255/visual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
- added link link_1; collision mesh filename=package://abb_irb6600_support/meshes/irb6600_225_255/collis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; visual mesh filename=package://abb_irb6600_support/meshes/irb6600_225_255/visual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
- added link link_1_mtr; collision mesh filename=package://abb_irb6600_support/meshes/irb6600_225_255/collis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; visual mesh filename=package://abb_irb6600_support/meshes/irb6600_225_255/visual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
- added link link_1_mtr2; collision mesh filename=package://abb_irb6600_support/meshes/irb6600_225_255/collis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; visual mesh filename=package://abb_irb6600_support/meshes/irb6600_225_255/visual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
- added link link_1_wt; collision mesh filename=package://abb_irb6600_support/meshes/irb6600_225_255/collis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; visual mesh filename=package://abb_irb6600_support/meshes/irb6600_225_255/visual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
- added link link_2; collision mesh filename=package://abb_irb6600_support/meshes/irb6600_225_255/collis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; visual mesh filename=package://abb_irb6600_support/meshes/irb6600_225_255/visual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
- added link link_3; collision mesh filename=package://abb_irb6600_support/meshes/irb6600_225_255/collis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; visual mesh filename=package://abb_irb6600_support/meshes/irb6600_225_255/visual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
- added link link_3_abb; collision mesh filename=package://abb_irb6600_support/meshes/irb6600_225_255/collis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; visual mesh filename=package://abb_irb6600_support/meshes/irb6600_225_255/visual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
- added link link_3_mtr; collision mesh filename=package://abb_irb6600_support/meshes/irb6600_225_255/collis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; visual mesh filename=package://abb_irb6600_support/meshes/irb6600_225_255/visual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
- added link link_3_mtr2; collision mesh filename=package://abb_irb6600_support/meshes/irb6600_225_255/collis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; visual mesh filename=package://abb_irb6600_support/meshes/irb6600_225_255/visual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
- added link link_4; collision mesh filename=package://abb_irb6600_support/meshes/irb6600_225_255/collis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; visual mesh filename=package://abb_irb6600_support/meshes/irb6600_225_255/visual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
- added link link_4_abb; collision mesh filename=package://abb_irb6600_support/meshes/irb6600_225_255/collis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; visual mesh filename=package://abb_irb6600_support/meshes/irb6600_225_255/visual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
- added link link_4_abb2; collision mesh filename=package://abb_irb6600_support/meshes/irb6600_225_255/collis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; visual mesh filename=package://abb_irb6600_support/meshes/irb6600_225_255/visual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
- added link link_5; collision mesh filename=package://abb_irb6600_support/meshes/irb6600_225_255/collis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; visual mesh filename=package://abb_irb6600_support/meshes/irb6600_225_255/visual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
- added link link_6; collision mesh filename=package://abb_irb6600_support/meshes/irb6600_225_255/collis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; visual mesh filename=package://abb_irb6600_support/meshes/irb6600_225_255/visual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
- added link tool0
Joints:
- added joint base_link-base: type fixed, parent base_link, child base, origin xyz=0 0 0 rpy=0 0 0
- added joint joint_1: type revolute, parent base_link, child link_1, origin xyz=0 0 0 rpy=0 0 0, axis 0 0 1, limit lower=-3.14159265 upper=3.14159265 effort=0 velocity=1.74532925
- added joint joint_1_mtr: type fixed, parent link_1, child link_1_mtr, origin xyz=0 0 0 rpy=0 0 0
- added joint joint_1_mtr2: type fixed, parent link_1, child link_1_mtr2, origin xyz=0 0 0 rpy=0 0 0
- added joint joint_1_wt: type fixed, parent link_1, child link_1_wt, origin xyz=0 0 0 rpy=0 0 0
- added joint joint_2: type revolute, parent link_1, child link_2, origin xyz=0.320 0 0.780 rpy=0 0 0, axis 0 1 0, limit lower=-1.13446401 upper=1.3962634 effort=0 velocity=1.57079633
- added joint joint_3: type revolute, parent link_2, child link_3, origin xyz=0 0 1.075 rpy=0 0 0, axis 0 1 0, limit lower=-3.14159265 upper=1.04719755 effort=0 velocity=1.57079633
- added joint joint_3_abb: type fixed, parent link_3, child link_3_abb, origin xyz=0 0 0 rpy=0 0 0
- added joint joint_3_mtr: type fixed, parent link_3, child link_3_mtr, origin xyz=0 0 0 rpy=0 0 0
- added joint joint_3_mtr2: type fixed, parent link_3, child link_3_mtr2, origin xyz=0 0 0 rpy=0 0 0
- added joint joint_4: type revolute, parent link_3, child link_4, origin xyz=0 0 0.2 rpy=0 0 0, axis 1 0 0, limit lower=-5.23598776 upper=5.23598776 effort=0 velocity=2.61799388
- added joint joint_4_abb: type fixed, parent link_4, child link_4_abb, origin xyz=0 0 0 rpy=0 0 0
- added joint joint_4_abb2: type fixed, parent link_4, child link_4_abb2, origin xyz=0 0 0 rpy=0 0 0
- added joint joint_5: type revolute, parent link_4, child link_5, origin xyz=1.142 0 0 rpy=0 0 0, axis 0 1 0, limit lower=-2.0943951 upper=2.0943951 effort=0 velocity=2.0943951
- added joint joint_6: type revolute, parent link_5, child link_6, origin xyz=0.2 0 0 rpy=0 0 0, axis 1 0 0, limit lower=-5.23598776 upper=5.23598776 effort=0 velocity=3.31612558
- added joint joint_6-tool0: type fixed, parent link_6, child tool0, origin xyz=0 0 0 rpy=0 1.57079632679 0
