Commit message: Further joint adjustments to prevent wrapup

File: abb_irb6600_support/urdf/irb6640_macro.xacro (robot description, xacro)
@@ -281,5 +281,5 @@
       <child link="${prefix}link_3" />
       <axis xyz="0 1 0" />
-      <limit lower="-3.14159265" upper="1.04719755" effort="0" velocity="1.57079633" />
+      <limit lower="-0.1" upper="1.04719755" effort="0" velocity="1.57079633" />
     </joint>
     <joint name="${prefix}joint_3_mtr" type="fixed">
@@ -303,5 +303,5 @@
       <child link="${prefix}link_4" />
       <axis xyz="1 0 0" />
-      <limit lower="-1.7" upper="1.7" effort="0" velocity="2.61799388" />
+      <limit lower="-1.6" upper="1.6" effort="0" velocity="2.61799388" />
     </joint>
     <joint name="${prefix}joint_4_abb" type="fixed">
@@ -320,5 +320,5 @@
       <child link="${prefix}link_5" />
       <axis xyz="0 1 0" />
-      <limit lower="-2.0943951" upper="2.0943951" effort="0" velocity="2.0943951" />
+      <limit lower="-2.0943951" upper="1.0" effort="0" velocity="2.0943951" />
     </joint>
     <joint name="${prefix}joint_6" type="revolute">
